File: Sundry.kicad_sch (KiCad schematic)
At the start: 24 parts, among them U1 74LVC1G74DP,125, U3 TLV3501AID

Commit message: Automatic save 2026-10-30 10:15:47
Parts:
- RV1: footprint Potentiometer_THT:Potentiometer_Bourns_3266X_Horizontal -> Potentiometer_THT:Potentiometer_Bourns_3266P_Horizontal
Changed lines of the file:
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@@
 			)
 		)
-		(property "Footprint" "Potentiometer_THT:Potentiometer_Bourns_3266X_Horizontal"
+		(property "Footprint" "Potentiometer_THT:Potentiometer_Bourns_3266P_Horizontal"
 			(at 133.35 76.2 0)
 			(hide yes)
