File: SonoLoad.kicad_pcb (KiCad board)
At the start: 4 copper layers, 85.6 x 54 mm, 43 parts, among them J1_PCD1 Conn_01x04, J2 Conn_01x07, J3 Conn_01x10, J5 Conn_01x08, P1 Conn_01x08, P1_LOAD1 Conn_01x04, P2 Conn_01x03, P2_LOAD1 Conn_01x04, P3 Conn_01x15, P6 Conn_01x15, U1 74LVC1G74DP,125, U2 Arduino_Nano_33_IoT_AllFuncti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, U3 TLV3501AID

Commit message: Automatic save 2026-10-29 21:00:33
Parts:
- added ?: , Common_Components:SonoLoad_GitHub_QR, F.Cu at (158.3, 121.0)

Commit message: Automatic save 2026-10-30 12:40:46
Parts:
- R2: value 100 kΩ -> 100kΩ
- RV1: footprint Potentiometer_THT:Potentiometer_Bourns_3266X_Horizontal -> Potentiometer_THT:Potentiometer_Bourns_3266P_Horizontal
- moved RV1 2.46 mm to (120.0, 101.1)
Routing:
- net /Sundry/OFFSET_BIAS: track 27.7 -> 29.5 mm
- net /ArduinoNano33_IOT/D06: track 69.3 -> 68.1 mm
Other:
- board text added: "SonoLoad Revision X1"
